Commit message: Update description package name

File: config/urdfs/amiga.urdf (robot description, URDF)
Before this commit: robot amiga, 60 links, 59 joints
Links:
- link amiga_arm_base_link: geometry collision mesh filename=package://ur_description/meshes/ur10e/collision/base.stl; visual mesh filename=package://ur_description/meshes/ur10e/visual/base.dae
- link amiga_arm_forearm_link: geometry collision mesh filename=package://ur_description/meshes/ur10e/collision/forearm.stl; visual mesh filename=package://ur_description/meshes/ur10e/visual/forearm.dae
- link amiga_arm_shoulder_link: geometry collision mesh filename=package://ur_description/meshes/ur10e/collision/shoulder.stl; visual mesh filename=package://ur_description/meshes/ur10e/visual/shoulder.dae
- link amiga_arm_upper_arm_link: geometry collision mesh filename=package://ur_description/meshes/ur10e/collision/upperarm.stl; visual mesh filename=package://ur_description/meshes/ur10e/visual/upperarm.dae
- link amiga_arm_wrist_1_link: geometry collision mesh filename=package://ur_description/meshes/ur10e/collision/wrist1.stl; visual mesh filename=package://ur_description/meshes/ur10e/visual/wrist1.dae
- link amiga_arm_wrist_2_link: geometry collision mesh filename=package://ur_description/meshes/ur10e/collision/wrist2.stl; visual mesh filename=package://ur_description/meshes/ur10e/visual/wrist2.dae
- link amiga_arm_wrist_3_link: geometry collision mesh filename=package://ur_description/meshes/ur10e/collision/wrist3.stl; visual mesh filename=package://ur_description/meshes/ur10e/visual/wrist3.dae
